File: kicad/mplex/mplex.kicad_pcb (KiCad board)
At the start: 4 copper layers, 53.5 x 76 mm, 14 parts, among them J101 PAL-1 Expansion Connector, SW101 PICO RESET, U101 74LVC245, U102 74LVC245, U103 Pico, U104 74LVC245, U105 74LVC245

Commit message: Trial of multiplexed code
Parts:
- removed R101: 1K, Resistor_THT:R_Axial_DIN0204_L3.6mm_D1.6mm_P5.08mm_Horizontal
Connections:
- U101 pad 19: /CS1 -> /~{ADDR_CE}
- U102 pad 1: /CDIR -> /DATA_DIR
- U102 pad 19: /CS3 -> /~{DATA_CE}
- U103 pad 11: /CDIR -> /LV8
- U103 pad 12: /CS1 -> /LV9
- U103 pad 14: /CS2 -> /LV10
- U103 pad 15: /CS3 -> /LV11
- U103 pad 16: unconnected-(U103-GPIO12-Pad16) -> /LV12
- U103 pad 17: unconnected-(U103-GPIO13-Pad17) -> /LV13
- U103 pad 19: unconnected-(U103-GPIO14-Pad19) -> /LV14
- U103 pad 20: unconnected-(U103-GPIO15-Pad20) -> /LV15
- U103 pad 21: unconnected-(U103-GPIO16-Pad21) -> /DATA_DIR
- U103 pad 22: unconnected-(U103-GPIO17-Pad22) -> /~{DATA_CE}
- U103 pad 24: unconnected-(U103-GPIO18-Pad24) -> /~{ADDR_CE}
- U103 pad 25: unconnected-(U103-GPIO19-Pad25) -> /~{CTL_CE}
- U104 pad 11: /LV7 -> /LV15
- U104 pad 12: /LV6 -> /LV14
- U104 pad 13: /LV5 -> /LV13
- U104 pad 14: /LV4 -> /LV12
- U104 pad 15: /LV3 -> /LV11
- U104 pad 16: /LV2 -> /LV10
- U104 pad 17: /LV1 -> /LV9
- U104 pad 18: /LV0 -> /LV8
- U104 pad 19: /CS2 -> /~{ADDR_CE}
- U105 pad 19: /CS4 -> /~{CTL_CE}
Routing:
- net /~{ADDR_CE}: track 0.00 -> 61.9 mm
- net /~{CTL_CE}: track 0.00 -> 41.2 mm
- net /CS3: track 34.4 -> 0.00 mm
- net /CDIR: track 30.0 -> 0.00 mm
- net /HVA8: track 44.6 -> 73.8 mm
- net /LV6: track 91.2 -> 62.5 mm
- net /HVA11: track 31.3 -> 59.7 mm
- net /CS1: track 27.4 -> 0.00 mm
- net /HVA6: track 83.4 -> 56.1 mm
- net /LV5: track 91.2 -> 64.0 mm
- net /LV7: track 89.8 -> 62.8 mm
- net /LV4: track 91.9 -> 64.9 mm
- net /LV3: track 91.2 -> 65.8 mm
- net /LV2: track 91.3 -> 66.2 mm
- net /HVA0: track 112.2 -> 90.2 mm
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Other:
- board text added: "MULTIPLEX (VER 3.0.0)"
- board text removed: "MULTIPLEX (VER 2.0.0)"
