File: kicad/mplex/mplex.kicad_sch (KiCad schematic)
At the start: 14 parts, among them J101 PAL-1 Expansion Connector, SW101 PICO RESET, U101 74LVC245, U102 74LVC245, U103 Pico, U104 74LVC245, U105 74LVC245

Commit message: Trial of multiplexed code
Parts:
- removed R101: 1K, Resistor_THT:R_Axial_DIN0204_L3.6mm_D1.6mm_P5.08mm_Horizontal, symbol Device:R_Small
Connections:
- net CS4 is gone; now on net GND: U105.19 (CE)
- net LV0: no longer U104.18 (B0)
- net LV1: no longer U104.17 (B1)
- net LV2: no longer U104.16 (B2)
- net LV3: no longer U104.15 (B3)
- net LV4: no longer U104.14 (B4)
- net LV5: no longer U104.13 (B5)
- net LV6: no longer U104.12 (B6)
- net LV7: no longer U104.11 (B7)
- net LV12: now reaches U103.16 (GPIO12)
- net LV12: now also U104.14 (B4)
- net LV13: now reaches U103.17 (GPIO13)
- net LV13: now also U104.13 (B5)
- net LV14: now reaches U103.19 (GPIO14)
- net LV14: now also U104.12 (B6)
- net LV15: now reaches U103.20 (GPIO15)
- net LV15: now also U104.11 (B7)
- net DATA_DIR: now reaches U103.21 (GPIO16)
- net DATA_DIR: now also U102.1 (A->B)
- net ~{DATA_CE}: now reaches U103.22 (GPIO17)
- net ~{DATA_CE}: now also U102.19 (CE)
- net ~{ADDR_CE}: now reaches U103.24 (GPIO18)
- net ~{ADDR_CE}: now also U101.19 (CE), U104.19 (CE)
- net CDIR renamed LV8
- net LV8: now also U104.18 (B0); no longer U102.1 (A->B)
- net CS1 renamed LV9
- net LV9: now also U104.17 (B1); no longer U101.19 (CE)
- net CS2 renamed LV10
- net LV10: now also U104.16 (B2); no longer U104.19 (CE)
- net CS3 renamed LV11
- net LV11: now also U104.15 (B3); no longer U102.19 (CE)
- no-connect marks 25 -> 29
Other:
- moved on the sheet: SW101
